Commit message: Possible Ergoaware changes

File: ur_description/urdf/ur_macro.xacro (robot description, xacro)
@@ -75,10 +75,10 @@
         </material>
       </visual>
-      <collision>
+      <!--collision>
         <origin xyz="0 0 0" rpy="0 0 ${pi}"/>
         <geometry>
           <mesh filename="${base_collision_mesh}"/>
         </geometry>
-      </collision>
+      </collision-->
       <xacro:cylinder_inertial radius="${base_inertia_radius}" length="${base_inertia_length}" mass="${base_mass}">
         <origin xyz="0 0 0" rpy="0 0 0" />
